File: Eagle Project/gba link.brd (EAGLE design)
At the start: 26 x 21 mm, 18 parts

Commit message: KiCad Start
Parts:
- U$1: device Catskulls_link_port:GBA-LINK-ALT -> Catskulls_link_portMirror:GBA-LINK-ALT
- moved U$1 27.5 mm to (-4.32, -14.3)
Routing:
- net N$1: track 23.6 -> 50.6 mm
- net N$2: track 43.5 -> 66.9 mm
Other:
- board size 26 x 21 mm -> 42.8 x 47.4 mm
Changed lines of the file:
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@@
 <board>
 <plain>
-<wire x1="-29.845" y1="23.495" x2="-29.845" y2="2.54" width="0.1524" layer="20"/>
-<wire x1="-29.845" y1="2.54" x2="-3.81" y2="2.54" width="0.1524" layer="20"/>
-<wire x1="-3.81" y1="2.54" x2="-3.81" y2="23.495" width="0.1524" layer="20"/>
-<wire x1="-3.81" y1="23.495" x2="-29.845" y2="23.495" width="0.1524" layer="20"/>
+<wire x1="-29.845" y1="23.495" x2="-29.845" y2="-23.368" width="0.1524" layer="20"/>
+<wire x1="-29.845" y1="-23.368" x2="12.954" y2="-22.86" width="0.1524" layer="20"/>
+<wire x1="12.954" y1="-22.86" x2="12.954" y2="24.003" width="0.1524" layer="20"/>
+<wire x1="12.954" y1="24.003" x2="-29.845" y2="23.495" width="0.1524" layer="20"/>
 </plain>
 <attributes>
@@
 </autorouter>
 <elements>
-<element name="U$1" library="Catskulls_link_port" package="GBA-LINK-ALT" value="GBA-LINKA" x="-19.05" y="8.89" smashed="yes"/>
+<element name="U$1" library="Catskulls_link_portMirror" package="GBA-LINK-ALT" value="GBA-LINKA" x="-4.318" y="-14.31" smashed="yes"/>
 <element name="CON" library="wirepad2" package="SMD1,27-2,54" package3d_urn="urn:adsk.eagle:package:30839/1" value="" x="-11.43" y="19.05" smashed="yes">
 <attribute name="NAME" x="-12.23" y="16.65" size="1.27" layer="25" rot="R90"/>
@@
 <contactref element="U$1" pad="VCC"/>
 <contactref element="+5V" pad="1"/>
-<wire x1="-17.12" y1="8.89" x2="-17.12" y2="12.7" width="0.508" layer="1"/>
+<wire x1="-2.388" y1="-14.31" x2="-17.12" y2="12.7" width="0.508" layer="1"/>
 <wire x1="-24.13" y1="12.7" x2="-24.13" y2="19.05" width="0.508" layer="1"/>
 <wire x1="-17.12" y1="12.7" x2="-24.13" y2="12.7" width="0.508" layer="1"/>
@@
 <contactref element="U$1" pad="GND"/>
 <wire x1="-15.24" y1="13.97" x2="-22.86" y2="13.97" width="0.508" layer="1"/>
-<wire x1="-20.98" y1="7.28" x2="-20.98" y2="5.08" width="0.508" layer="1"/>
+<wire x1="-6.248" y1="-15.92" x2="-20.98" y2="5.08" width="0.508" layer="1"/>
 <wire x1="-20.98" y1="5.08" x2="-20.98" y2="3.81" width="0.508" layer="1"/>
 <wire x1="-20.98" y1="3.81" x2="-12.7" y2="3.81" width="0.508" layer="1"/>
