File: Eagle Project/gba link.sch (EAGLE design)
At the start: 18 parts

Commit message: KiCad Start
Parts:
- U$1: device Catskulls_link_port:GBA-LINKA -> Catskulls_link_portMirror:GBA-LINKA
Changed lines of the file:
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@@
 </classes>
 <parts>
-<part name="U$1" library="Catskulls_link_port" deviceset="GBA-LINK" device="A"/>
+<part name="U$1" library="Catskulls_link_portMirror" deviceset="GBA-LINK" device="A"/>
 <part name="CON" library="wirepad2" deviceset="SMD2" device="" package3d_urn="urn:adsk.eagle:package:30839/1"/>
 <part name="DM" library="wirepad2" deviceset="SMD2" device="" package3d_urn="urn:adsk.eagle:package:30839/1"/>
